File: payload/hardware/CSUF-USLI-payload-2026/CSUF-USLI-payload-2026.kicad_sch (KiCad schematic)
At the start: 25 parts, among them M1 Motor_Servo, U1 DEV-16771, U2 GPS6MV2, U3 MPU6050, U4 Adafruit BMP390, U5 RYLR896, U6 Generic RS485 to UART, U7 DF Robot EC and pH Placeholder

Commit message: CDR Schematic done
Parts:
- removed C1, C2: 0.1 uF, symbol Device:C
- removed C3, C4: 100 uF, symbol Device:C_Polarized
- added C1: 0.1 uF, symbol Device:C_Small
- added C2: 1 uF, symbol Device:C_Small
- added C3: 10 uF, symbol Device:C_Small
- added C4: 100 uF, symbol Device:C_Small
- added D2: 25GA370 Brushed DC Motor, symbol L298N Concept:12V_Drill
- added D3: LED, symbol Device:LED
- added H1, H2, H3, H4: MountingHole, symbol Mechanical:MountingHole
- added J1: TD3 Connection, symbol Connector:Screw_Terminal_01x02
- added L2: L298N Motor Driver, symbol L298N Concept:L298N
- added M2, M3, M4: Motor_Servo, symbol Motor:Motor_Servo
- added Q1: IRLZ44N, symbol Simulation_SPICE:NMOS
- added R1: 1.5k, symbol Device:R_US
- added R2: 330, symbol Device:R_US
- added R3: 10k, symbol Device:R_US
- added SW1: Screw Switch, symbol Switch:SW_SPST
- added U8: RYLR896, symbol RYLR896:RYLR896
- BT1: value 13.3v Battery Cell -> 11.1v Lipo Battery
- D1: value Drill -> Warrior 12 V Brushed DC Motor
- G3, G4: value 12V Motor -> UXCELL 12V Brushed
- L1: value L298N DualDC Motor Driver -> L298N Dual Motor Driver
- L3: value Generic Motor Driver -> HiLetGo BTS7690 Motor Driver
- U4: value Adafruit BMP390 -> Adafruit BMP280
- U6: value Generic RS485 to UART -> RS485 to UART
- U7: value DF Robot EC and pH Placeholder -> Halisense Soil Sensor
Connections:
- net +3.3V: now also C7.1, U8.1 (VDD)
- net +5V: now also J1.1 (Pin_1); no longer C7.1, U1.VIN
- net BUZZ_P: now also U1.32 (OUT1B); no longer U1.31 (CTX3)
- net DRILL_IN1: now also U1.41 (A17)
- net DRILL_IN2: now also U1.40 (A16)
- net GND: now also C1.2, C2.2, C3.2, C4.2, L2. (Input1), M2.3 (-), M3.3 (-), M4.3 (-), Q1.3 (S), R1.2, R3.1, U8.6 (GND)
- net ROVER_IN1: now also U1.27 (A13)
- net ROVER_IN2: now also U1.26 (A12)
- net ROVER_IN3: now also U1.25 (A11)
- net ROVER_IN4: now also U1.24 (A10)
- net LEG_PWM1: now reaches U1.15 (A1)
- net LEG_PWM1: now also M2.1 (PWM)
- net LEG_PWM2: now reaches U1.16 (A2)
- net LEG_PWM2: now also M3.1 (PWM)
- net LEG_PWM3: now reaches U1.17 (A3)
- net LEG_PWM3: now also M4.1 (PWM)
- net IN_RYLR896_RX: now reaches U1.20 (A6)
- net IN_RYLR896_RX: now also U8.3 (RXD)
- net IN_RYLR896_TX: now reaches U1.21 (A7)
- net IN_RYLR896_TX: now also U8.4 (TXD)
- net TD3: now reaches U1.33 (MCLK2)
- net TD3: now also R2.1
- net CHASSIS_IN2: now reaches U1.38 (A14)
- net CHASSIS_IN2: now also L2. (Input1)
- net CHASSIS_IN1: now reaches U1.39 (A15)
- net CHASSIS_IN1: now also L2. (Input1)
- net at U1.5V: now also C1.1, C2.1, C3.1, C4.1
- removed net +13.3V: BT1.1 (+), L1. (Input4), L3. (Input1), M1.2 (+)
- net LEG_PWM renamed LEG_PWM0
- net RYLR896_RX renamed OUT_RYLR896_RX
- net RYLR896_TX renamed OUT_RYLR896_TX
- new net: D1. (M2), L3. (Input1)
- new net: J1.2 (Pin_2), Q1.1 (D)
- new net: D2. (M2), L2. (Input1) (x2)
- new net: Q1.2 (G), R2.2, R3.2
- new net: BT1.1 (+), SW1.1 (A)
- new net: G3. (M2), L1. (Input4)
- new net: G4. (M2), L1. (Input4)
- new net: D3.1 (K), R1.1
- new net +11.1V: D3.2 (A), L1. (Input4), L2. (Input1), L3. (Input1), M1.2 (+), M2.2 (+), M3.2 (+), M4.2 (+), SW1.2 (B)
Other:
- note added: "D.R.O.P"
- note added: "Flipping Subsystem"
- note added: "Mechanical"
- note added: "Rover Control Subsystem"
- note added: "TD3 Interface"
- note removed: "Legs Subsystem"
- note removed: "Rover Subsystem"
- note removed: "UTG Payload"
- moved on the sheet: BT1, BT2, BZ1, C5, C9, D1, L3, M1, U1, U3, U5, U6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

Commit message: Current VDF
Parts:
- removed G3, G4: UXCELL 12V Brushed, symbol Generic Devices:12V_Motor
- removed L1: L298N Dual Motor Driver, symbol L298N Concept:L298N
- added D4, D5: D, symbol Device:D
- added J2: 11.1V Input, symbol Connector:Screw_Terminal_01x02
- added J3: 8.4V Output, symbol Connector:Screw_Terminal_01x02
- added M5: R UXCELL 12V Brushed, symbol Motor:Motor_DC_ALT
- added M6: L UXCELL 12V Brushed, symbol Motor:Motor_DC_ALT
- added Q2, Q3: IRLZ44N, symbol Simulation_SPICE:NMOS
- added R4, R5: 3.3k, symbol Device:R_US
Connections:
- net +11.1V: now also D4.1 (K), D5.1 (K), J2.2 (Pin_2), M5.1 (+), M6.1 (+); no longer M1.2 (+), M2.2 (+), M3.2 (+), M4.2 (+)
- net GND: now also J2.1 (Pin_1), J3.2 (Pin_2), Q2.3 (S), Q3.3 (S)
- net ROVER_IN1: now also R4.1
- net ROVER_IN2: now also R5.1
- net ROVER_IN3: no longer names the net of U1.25 (A11)
- net ROVER_IN4: no longer names the net of U1.24 (A10)
- new net: D1. (M2), L3. (Input1)
- new net: D4.2 (A), M6.2 (-), Q2.1 (D)
- new net: Q2.2 (G), R4.2
- new net: D2. (M2), L2. (Input1)
- new net: Q3.2 (G), R5.2
- new net: D5.2 (A), M5.2 (-), Q3.1 (D)
- new net +8.4V: J3.1 (Pin_1), M1.2 (+), M2.2 (+), M3.2 (+), M4.2 (+)
Other:
- moved on the sheet: BT1, BT2, D3, R1, SW1
