File: payload/hardware/VDF/Sensor_Sled/Sensor_Sled.kicad_pcb (KiCad board)
At the start: 2 copper layers, 40.6 x 124.5 mm, 21 parts, among them J1 TD3 Connection, J2 Servo JST, J3 Chassis JST, J4 Drill x Rover JST, J5 Soil JST, J6 Reserve JST, J7 RYLR896 JST, J8 GPS x Power JST, Q1 IRLZ44N, U1 DEV-16771, U3 MPU6050, U4 Adafruit BMP280

Commit message: printed stuff
Connections:
- J5 pad 1: +3V3 -> +5V
Routing:
- net +5V: track 7.50 -> 67.2 mm
- net GND: track 173.7 -> 158.1 mm
- net +3V3: track 209.9 -> 201.3 mm
Changed lines of the file:
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@@
 			(remove_unused_layers no)
 			(roundrect_rratio 0.208333)
-			(net 5 "+3V3")
+			(net 3 "+5V")
 			(pinfunction "Pin_1")
 			(pintype "passive")
@@
 			(keep_text_aligned yes)
 		)
-		(gr_text "12.7000 mm"
+		(gr_text "500.0000 mils"
 			(at 115.57 163.3 0)
 			(layer "Eco1.User")
@@
 			(keep_text_aligned yes)
 		)
-		(gr_text "124.4600 mm"
+		(gr_text "4900.0000 mils"
 			(at 161.39349 92.71 90)
 			(layer "Eco1.User")
@@
 			(keep_text_aligned yes)
 		)
-		(gr_text "27.9400 mm"
+		(gr_text "1100.0000 mils"
 			(at 135.89 168.38 0)
 			(layer "Eco1.User")
@@
 			(keep_text_aligned yes)
 		)
-		(gr_text "53.3400 mm"
+		(gr_text "2100.0000 mils"
 			(at 94.72 128.27 90)
 			(layer "Eco1.User")
@@
 	)
 	(segment
-		(start 118.485 63.119)
-		(end 125.758 63.119)
-		(width 0.2)
-		(layer "B.Cu")
-		(net 2)
-	)
-	(segment
 		(start 124.1264 39.0144)
 		(end 120.65 39.0144)
@@
 	)
 	(segment
-		(start 112.564 69.04)
-		(end 118.485 63.119)
-		(width 0.2)
-		(layer "B.Cu")
-		(net 2)
-	)
-	(segment
 		(start 129.02 142.748)
 		(end 129.02 149.338)
@@
 	)
 	(segment
+		(start 116.63349 71.67051)
+		(end 112.564 75.74)
+		(width 2.000001)
+		(layer "B.Cu")
+		(net 3)
+	)
+	(segment
+		(start 135.89 39.0144)
+		(end 133.0836 36.208)
+		(width 2.000001)
+		(layer "B.Cu")
+		(net 3)
+	)
+	(segment
+		(start 133.0836 36.208)
+		(end 119.93349 36.208)
+		(width 2.000001)
+		(layer "B.Cu")
+		(net 3)
+	)
+	(segment
+		(start 119.93349 36.208)
+		(end 116.63349 39.508)
+		(width 2.000001)
+		(layer "B.Cu")
+		(net 3)
+	)
+	(segment
+		(start 116.63349 39.508)
+		(end 116.63349 71.67051)
+		(width 2.000001)
+		(layer "B.Cu")
+		(net 3)
+	)
+	(segment
 		(start 143.764 40.894)
 		(end 145.415 39.243)
@@
 	)
 	(segment
-		(start 113.7296 74.5744)
-		(end 112.564 75.74)
-		(width 1)
-		(layer "F.Cu")
-		(net 5)
-	)
-	(segment
 		(start 124.408 121.158)
 		(end 124.258 121.308)
@@
 		(width 1)
 		(layer "F.Cu")
-		(net 5)
-	)
-	(segment
-		(start 120.65 74.5744)
-		(end 113.7296 74.5744)
-		(width 1)
-		(layer "F.Cu")
